Commit message: modi thruster config as X4omni

File: src/robot/urdf/robot.urdf_modified.urdf (robot description, URDF)
Before this commit: robot njord_asv, 6 links, 5 joints
Links:
- added link thruster_FL_link; visual cylinder length=0.113 radius=0.1
- added link thruster_FR_link; visual cylinder length=0.113 radius=0.1
- added link thruster_RL_link; visual cylinder length=0.113 radius=0.1
- added link thruster_RR_link; visual cylinder length=0.113 radius=0.1
Joints:
- added joint thruster_FL_joint: type fixed, parent base_link, child thruster_FL_link, origin xyz=0.353553 0.353553 0.0 rpy=0 0 -0.785398
- added joint thruster_FR_joint: type fixed, parent base_link, child thruster_FR_link, origin xyz=0.353553 -0.353553 0.0 rpy=0 0 0.785398
- added joint thruster_RL_joint: type fixed, parent base_link, child thruster_RL_link, origin xyz=-0.353553 0.353553 0.0 rpy=0 0 -2.35619
- added joint thruster_RR_joint: type fixed, parent base_link, child thruster_RR_link, origin xyz=-0.353553 -0.353553 0.0 rpy=0 0 2.35619
