Commit message: modi odom frame and add manual

File: src/robot/urdf/robot.urdf.xacro (robot description, xacro)
@@ -52,5 +52,5 @@
     <origin xyz="${lidar_x} ${lidar_y} ${lidar_z}" rpy="0 0 0"/>
   </joint>
-  <link name="imu_link">
+  <link name="wit_imu_frame">
     <visual>
       <geometry>
@@ -62,7 +62,7 @@
     </visual>
   </link>
-  <joint name="imu_joint" type="fixed">
+  <joint name="wit_imu_joint" type="fixed">
     <parent link="base_link"/>
-    <child link="imu_link"/>
+    <child link="wit_imu_frame"/>
     <origin xyz="${imu_x} ${imu_y} ${imu_z}" rpy="0 0 0"/>
   </joint>
@@ -82,15 +82,17 @@
     <origin xyz="${gnss1_x} ${gnss1_y} ${gnss1_z}" rpy="0 0 0"/>
   </joint>
-  <link name="gnss_sub_link">
-     <visual>
+  <link name="rzs_frame">
+    <visual>
       <geometry>
         <cylinder radius="0.08" length="0.05"/>
       </geometry>
-      <material name="white"/>
+      <material name="white">
+        <color rgba="1.0 1.0 1.0 1.0"/>
+      </material>
     </visual>
   </link>
-  <joint name="gnss_sub_joint" type="fixed">
+  <joint name="rzs_joint" type="fixed">
     <parent link="base_link"/>
-    <child link="gnss_sub_link"/>
+    <child link="rzs_frame"/>
     <origin xyz="${gnss2_x} ${gnss2_y} ${gnss2_z}" rpy="0 0 0"/>
   </joint>

Commit message: add and modi nav2_params etc

File: src/robot/urdf/robot.urdf.xacro (robot description, xacro)
@@ -16,10 +16,4 @@
   <xacro:property name="gnss2_y" value="-0.4" />
   <xacro:property name="gnss2_z" value="1.0" />
-  <link name="base_footprint"/>
-  <joint name="base_joint" type="fixed">
-    <parent link="base_footprint"/>
-    <child link="base_link"/>
-    <origin xyz="0 0 ${base_height/2}" rpy="0 0 0"/>
-  </joint>
   <link name="base_link">
     <visual>

File: src/robot/urdf/robot.urdf_modified.urdf (robot description, URDF)
Before this commit: robot njord_asv, 6 links, 5 joints
Links:
- removed link base_footprint
Joints:
- removed joint base_joint

Commit message: task3: buoy_obstacle_publisher pkg, field_boundary, task3 nav2 params, robot_radius=1.4m, imu_link TF fix, both buoy sets always published

File: src/robot/urdf/robot.urdf.xacro (robot description, xacro)
@@ -1,7 +1,7 @@
 <?xml version="1.0"?>
 <robot name="njord_asv" xmlns:xacro="http://ros.org/wiki/xacro">
-  <xacro:property name="base_width" value="1.0" />
-  <xacro:property name="base_length" value="1.5" />
-  <xacro:property name="base_height" value="0.5" />
+  <xacro:property name="base_width" value="1.85" />
+  <xacro:property name="base_length" value="2.0" />
+  <xacro:property name="base_height" value="1.2" />
   <xacro:property name="lidar_x" value="0.5" />
   <xacro:property name="lidar_y" value="0.0" />
@@ -61,4 +61,11 @@
     <origin xyz="${imu_x} ${imu_y} ${imu_z}" rpy="0 0 0"/>
   </joint>
+  <!-- imu_link: alias used by sensor_noise_simulator and EKF -->
+  <link name="imu_link"/>
+  <joint name="imu_link_joint" type="fixed">
+    <parent link="base_link"/>
+    <child link="imu_link"/>
+    <origin xyz="0.0 0.0 0.2" rpy="0 0 0"/>
+  </joint>
   <link name="gnss_link">
     <visual>

File: src/robot/urdf/robot.urdf_modified.urdf (robot description, URDF)
Before this commit: robot njord_asv, 5 links, 4 joints
Links:
- removed link gnss_sub_link
- added link rzs_frame; visual cylinder length=0.05 radius=0.08
- added link wit_imu_frame; visual box size=0.05 0.05 0.02
- link base_link: mass 1. -> None; geometry collision box size=2.0 1.85 1.2; visual box size=2.0 1.85 1.2
- link gnss_link: mass 1. -> None
- link imu_link: mass 1. -> None; geometry 
- link livox_frame: mass 1. -> None
Joints:
- removed joint gnss_sub_joint
- removed joint imu_joint
- added joint imu_link_joint: type fixed, parent base_link, child imu_link, origin xyz=0.0 0.0 0.2 rpy=0 0 0
- added joint rzs_joint: type fixed, parent base_link, child rzs_frame, origin xyz=-0.5 -0.4 1.0 rpy=0 0 0
- added joint wit_imu_joint: type fixed, parent base_link, child wit_imu_frame, origin xyz=0.0 0.0 0.2 rpy=0 0 0

Commit message: fix: route thruster control through urdf-aware driver

File: src/robot/urdf/robot.urdf.xacro (robot description, xacro)
@@ -16,4 +16,24 @@
   <xacro:property name="gnss2_y" value="-0.4" />
   <xacro:property name="gnss2_z" value="1.0" />
+  <xacro:property name="thruster_front_x" value="0.1803" />
+  <xacro:property name="thruster_rear_x" value="-0.1803" />
+  <xacro:property name="thruster_right_y" value="-0.2500" />
+  <xacro:property name="thruster_left_y" value="0.2500" />
+  <xacro:property name="thruster_z" value="-0.1" />
+  <xacro:macro name="thruster_link" params="name x y z">
+    <link name="${name}">
+      <visual>
+        <geometry>
+          <cylinder radius="0.04" length="0.16"/>
+        </geometry>
+        <material name="black"/>
+      </visual>
+    </link>
+    <joint name="${name}_joint" type="fixed">
+      <parent link="base_link"/>
+      <child link="${name}"/>
+      <origin xyz="${x} ${y} ${z}" rpy="0 0 0"/>
+    </joint>
+  </xacro:macro>
   <link name="base_footprint"/>
   <joint name="base_joint" type="fixed">
@@ -95,3 +115,7 @@
     <origin xyz="${gnss2_x} ${gnss2_y} ${gnss2_z}" rpy="0 0 0"/>
   </joint>
+  <xacro:thruster_link name="thruster_FR" x="${thruster_front_x}" y="${thruster_right_y}" z="${thruster_z}"/>
+  <xacro:thruster_link name="thruster_FL" x="${thruster_front_x}" y="${thruster_left_y}" z="${thruster_z}"/>
+  <xacro:thruster_link name="thruster_RR" x="${thruster_rear_x}" y="${thruster_right_y}" z="${thruster_z}"/>
+  <xacro:thruster_link name="thruster_RL" x="${thruster_rear_x}" y="${thruster_left_y}" z="${thruster_z}"/>
 </robot>

File: src/robot/urdf/robot.urdf_modified.urdf (robot description, URDF)
Before this commit: robot njord_asv, 6 links, 5 joints
Links:
- added link thruster_FL; visual cylinder length=0.16 radius=0.04
- added link thruster_FR; visual cylinder length=0.16 radius=0.04
- added link thruster_RL; visual cylinder length=0.16 radius=0.04
- added link thruster_RR; visual cylinder length=0.16 radius=0.04
Joints:
- added joint thruster_FL_joint: type fixed, parent base_link, child thruster_FL, origin xyz=0.1803 0.2500 -0.1 rpy=0 0 0
- added joint thruster_FR_joint: type fixed, parent base_link, child thruster_FR, origin xyz=0.1803 -0.2500 -0.1 rpy=0 0 0
- added joint thruster_RL_joint: type fixed, parent base_link, child thruster_RL, origin xyz=-0.1803 0.2500 -0.1 rpy=0 0 0
- added joint thruster_RR_joint: type fixed, parent base_link, child thruster_RR, origin xyz=-0.1803 -0.2500 -0.1 rpy=0 0 0

Commit message: Fix task3 sim navigation flow

File: src/robot/urdf/robot.urdf.xacro (robot description, xacro)
@@ -36,10 +36,4 @@
     </joint>
   </xacro:macro>
-  <link name="base_footprint"/>
-  <joint name="base_joint" type="fixed">
-    <parent link="base_footprint"/>
-    <child link="base_link"/>
-    <origin xyz="0 0 ${base_height/2}" rpy="0 0 0"/>
-  </joint>
   <link name="base_link">
     <visual>

File: src/robot/urdf/robot.urdf_modified.urdf (robot description, URDF)
Before this commit: robot njord_asv, 10 links, 9 joints
Links:
- removed link base_footprint
Joints:
- removed joint base_joint

Commit message: feat: integrate advanced navigation spatial ins

File: src/robot/urdf/robot.urdf.xacro (robot description, xacro)
@@ -87,4 +87,11 @@
     <origin xyz="${imu_x} ${imu_y} ${imu_z}" rpy="0 0 0"/>
   </joint>
+  <!-- Placeholder Spatial extrinsics. Measure and replace before tuning fusion. -->
+  <link name="spatial_link"/>
+  <joint name="spatial_joint" type="fixed">
+    <parent link="base_link"/>
+    <child link="spatial_link"/>
+    <origin xyz="0 0 0" rpy="0 0 0"/>
+  </joint>
   <link name="gnss_link">
     <visual>
