Commit message: Apply nominal upside-down LiDAR mount (roll=pi) in URDF only
- robot.urdf.xacro: add lidar_roll/pitch/yaw xacro properties
  (default roll=pi, nominal, needs on-vessel verification) and use
  them in the livox_frame joint rpy
- robot.urdf_modified.urdf: same joint rpy set to "3.14159265 0 0"
- Comments state this joint is the single place the inversion is
  applied; perception nodes rely on TF only

Co-Authored-By: Claude Fable 5 <noreply@anthropic.com>

File: src/robot/urdf/robot.urdf.xacro (robot description, xacro)
@@ -7,4 +7,13 @@
   <xacro:property name="lidar_y" value="0.0" />
   <xacro:property name="lidar_z" value="0.8" />
+  <!--
+    NOMINAL 180-deg roll for upside-down Mid360 mounting - MEASURE and update
+    before trusting perception/GLIM; this URDF is the ONLY inversion
+    correction point; do not re-rotate in nodes. Perception nodes must simply
+    transform livox_frame -> base_link via TF.
+  -->
+  <xacro:property name="lidar_roll" value="3.14159265358979" />
+  <xacro:property name="lidar_pitch" value="0" />
+  <xacro:property name="lidar_yaw" value="0" />
   <xacro:property name="imu_x" value="0.0" />
   <xacro:property name="imu_y" value="0.0" />
@@ -70,5 +79,5 @@
     <parent link="base_link"/>
     <child link="livox_frame"/>
-    <origin xyz="${lidar_x} ${lidar_y} ${lidar_z}" rpy="0 0 0"/>
+    <origin xyz="${lidar_x} ${lidar_y} ${lidar_z}" rpy="${lidar_roll} ${lidar_pitch} ${lidar_yaw}"/>
   </joint>
   <link name="imu_link">

File: src/robot/urdf/robot.urdf_modified.urdf (robot description, URDF)
Before this commit: robot njord_asv, 10 links, 9 joints
Joints:
- joint lidar_joint: origin xyz=0.5 0.0 0.8 rpy=0 0 0 -> xyz=0.5 0.0 0.8 rpy=3.14159265358979 0 0
