Commit message: launch理解、整備

File: src/robot/urdf/robot.urdf.xacro (robot description, xacro)
@@ -70,5 +70,7 @@
     <parent link="base_link"/>
     <child link="livox_frame"/>
-    <origin xyz="${lidar_x} ${lidar_y} ${lidar_z}" rpy="0 0 0"/>
+    <!-- The MID-360 is mounted upside down: preserve its origin while
+         rotating its frame 180 degrees around the vehicle X axis. -->
+    <origin xyz="${lidar_x} ${lidar_y} ${lidar_z}" rpy="3.141592653589793 0 0"/>
   </joint>
   <link name="imu_link">

File: src/robot/urdf/robot.urdf_modified.urdf (robot description, URDF)
Before this commit: robot njord_asv, 10 links, 9 joints
Joints:
- joint lidar_joint: origin xyz=0.5 0.0 0.8 rpy=0 0 0 -> xyz=0.5 0.0 0.8 rpy=3.141592653589793 0 0

Commit message: zikken suruzo

File: src/robot/urdf/robot.urdf.xacro (robot description, xacro)
@@ -13,5 +13,5 @@
   <xacro:property name="gnss1_y" value="0.4" />
   <xacro:property name="gnss1_z" value="1.0" />
-  <xacro:property name="gnss2_x" value="-0.5" />
+  <xacro:property name="gnss2_x" value="0.5" />
   <xacro:property name="gnss2_y" value="-0.4" />
   <xacro:property name="gnss2_z" value="1.0" />
@@ -57,4 +57,11 @@
     </collision>
   </link>
+  <!-- ZED2i left camera optical-origin frame, rigidly mounted at the bow. -->
+  <link name="zed2i_left_camera_frame"/>
+  <joint name="zed2i_left_camera_joint" type="fixed">
+    <parent link="base_link"/>
+    <child link="zed2i_left_camera_frame"/>
+    <origin xyz="0.48 0 0.47" rpy="0 0 0"/>
+  </joint>
   <link name="livox_frame">
     <visual>

Commit message: Make local EKF an explicit fallback

File: src/robot/urdf/robot.urdf.xacro (robot description, xacro)
@@ -57,4 +57,19 @@
     <child link="zed2i_left_camera_frame"/>
     <origin xyz="0.48 0 0.47" rpy="0 0 0"/>
+  </joint>
+  <!-- The right imager is 15 cm to starboard of the left imager. -->
+  <link name="zed2i_right_camera_frame"/>
+  <joint name="zed2i_right_camera_joint" type="fixed">
+    <parent link="zed2i_left_camera_frame"/>
+    <child link="zed2i_right_camera_frame"/>
+    <origin xyz="0 -0.15 0" rpy="0 0 0"/>
+  </joint>
+  <!-- Rear camera: 60 cm aft of the ZED2i stereo centre, facing aft.
+       Relative to the left imager, the stereo centre is 7.5 cm starboard. -->
+  <link name="back_cam_link"/>
+  <joint name="back_cam_joint" type="fixed">
+    <parent link="zed2i_left_camera_frame"/>
+    <child link="back_cam_link"/>
+    <origin xyz="-0.60 -0.075 0" rpy="0 0 3.141592653589793"/>
   </joint>
   <link name="livox_frame">
